File: KiCad/Versie2/Versie2.kicad_pcb (KiCad board)
At the start: 2 copper layers, 60 x 50 mm, 80 parts, among them IC1 AP9221SA-CC-HAC-7, IC2 ISL91107IRTNZ-T7A, J1 Leftover, J2 USB_C_Receptacle_USB3.0, J3 JTAG, J4 Programmer, J5 SPI, J6 I2C, J7 BOOT, J8 Screw_Terminal_01x02, J9 Screw_Terminal_01x02, Q1 Q_NMOS_GSD, Q2 Q_NMOS_GSD, Q3 Q_NMOS_GSD, Q4 Q_NMOS_GSD, U1 ESP32-WROOM-32, U2 MCP73831T-2ATI_MC, Y1 32.768kHz

Commit message: KiCad PCB IC Layout
Parts:
- removed AC1: BNO080, Versie1_FootprintLib:BNO080
- removed J5: SPI, Connector_PinHeader_2.54mm:PinHeader_1x08_P2.54mm_Vertical
- removed JP1, JP2: Jumper_NO_Small, Jumper:SolderJumper-2_P1.3mm_Open_Pad1.0x1.5mm
- removed JP3, JP6: SolderJumper_2_Open, Jumper:SolderJumper-2_P1.3mm_Open_Pad1.0x1.5mm
- removed JP4, JP5, JP7: SolderJumper_3_Open, Jumper:SolderJumper-3_P1.3mm_Open_Pad1.0x1.5mm
- removed Y1: 32.768kHz, Crystal:Crystal_SMD_3215-2Pin_3.2x1.5mm
- added C15: 1uF, Capacitor_SMD:C_0603_1608Metric, F.Cu at (158.4, 161.2)
- added C16: 100nF, Capacitor_SMD:C_0603_1608Metric, F.Cu at (126.4, 126.4)
- added C17: 1uF, Capacitor_SMD:C_0603_1608Metric, F.Cu at (158.4, 164.2)
- added C18: 100nF, Capacitor_SMD:C_0603_1608Metric, F.Cu at (158.4, 162.7)
- added C19: 100nF, Capacitor_SMD:C_0603_1608Metric, F.Cu at (158.4, 165.7)
- added J10: Screw_Terminal_01x02, TerminalBlock_TE-Connectivity:TerminalBlock_TE_282834-2_1x02_P2.54mm_Horizontal, F.Cu at (123.5, 90.8)
- added J11: Screw_Terminal_01x02, TerminalBlock_TE-Connectivity:TerminalBlock_TE_282834-2_1x02_P2.54mm_Horizontal, F.Cu at (103.6, 74.4)
- added Q10: Q_NMOS_GSD, Package_TO_SOT_SMD:SOT-23, F.Cu at (103.6, 68.9)
- added Q5: Q_NMOS_GSD, Package_TO_SOT_SMD:SOT-23, F.Cu at (148.0, 158.7)
- added Q6: Q_NMOS_GSD, Package_TO_SOT_SMD:SOT-23, F.Cu at (151.5, 158.7)
- added Q7: Q_NMOS_GSD, Package_TO_SOT_SMD:SOT-23, F.Cu at (144.4, 158.7)
- added Q8: Q_NMOS_GSD, Package_TO_SOT_SMD:SOT-23, F.Cu at (155.1, 158.7)
- added Q9: Q_NMOS_GSD, Package_TO_SOT_SMD:SOT-23, F.Cu at (117.8, 120.3)
- added R28: 2.2k, Resistor_SMD:R_0603_1608Metric, F.Cu at (144.4, 156.2)
- added R29: 2.2k, Resistor_SMD:R_0603_1608Metric, F.Cu at (155.1, 156.2)
- added R30: 1k, Resistor_SMD:R_0603_1608Metric, F.Cu at (189.2, 101.6)
- added R31: 1k, Resistor_SMD:R_0603_1608Metric, F.Cu at (185.9, 101.6)
- added R32: 10k, Resistor_SMD:R_0603_1608Metric, F.Cu at (113.3, 130.9)
- added U3: NE555DR, Package_SO:SOIC-8_3.9x4.9mm_P1.27mm, F.Cu at (115.4, 147.8)
- added U4: NE555DR, Package_SO:SOIC-8_3.9x4.9mm_P1.27mm, F.Cu at (132.7, 147.9)
- added U5: MIC5366-1.8YC5-TR, Package_TO_SOT_SMD:SOT-353_SC-70-5, F.Cu at (158.6, 158.8)
- added U6: ICM-20948, Sensor_Motion:InvenSense_QFN-24_3x3mm_P0.4mm, F.Cu at (154.6, 164.2)
- C1, C12, C13, C14, C2, C3, C4, C5, C7, C8, C9: footprint Capacitor_SMD:C_0603_1608Metric_Pad1.05x0.95mm_HandSolder -> Capacitor_SMD:C_0603_1608Metric
- C10: value 22pF -> 10nF; footprint Capacitor_SMD:C_0603_1608Metric_Pad1.05x0.95mm_HandSolder -> Capacitor_SMD:C_0603_1608Metric
- C11: value 22pF -> 1uF; footprint Capacitor_SMD:C_0603_1608Metric_Pad1.05x0.95mm_HandSolder -> Capacitor_SMD:C_0603_1608Metric
- C6: value 100nF -> 10nF; footprint Capacitor_SMD:C_0603_1608Metric_Pad1.05x0.95mm_HandSolder -> Capacitor_SMD:C_0603_1608Metric
- J1: value Leftover -> Micro_SD_Card; footprint Connector_PinHeader_2.54mm:PinHeader_1x04_P2.54mm_Vertical -> Connector_Card:microSD_HC_Molex_104031-0811
- J6: value I2C -> Screw_Terminal_01x02; footprint Connector_PinHeader_2.54mm:PinHeader_1x08_P2.54mm_Vertical -> TerminalBlock_TE-Connectivity:TerminalBlock_TE_282834-2_1x02_P2.54mm_Horizontal
- J7: value BOOT -> Screw_Terminal_01x02; footprint Connector_PinHeader_2.54mm:PinHeader_1x01_P2.54mm_Vertical -> TerminalBlock_TE-Connectivity:TerminalBlock_TE_282834-2_1x02_P2.54mm_Horizontal
- JP8, JP9: moved to F.Cu
- R1, R10, R12, R13, R15, R16, R17, R19, R2, R22, R23, R25, R26, R27, R3, R4, R5, R6, R7, R8, R9: footprint Resistor_SMD:R_0603_1608Metric_Pad1.05x0.95mm_HandSolder -> Resistor_SMD:R_0603_1608Metric
- R11, R14: value 10k -> 180k; footprint Resistor_SMD:R_0603_1608Metric_Pad1.05x0.95mm_HandSolder -> Resistor_SMD:R_0603_1608Metric
- R18, R20: value 4.7k -> 2.2k; footprint Resistor_SMD:R_0603_1608Metric_Pad1.05x0.95mm_HandSolder -> Resistor_SMD:R_0603_1608Metric
- R21: value 10k -> 2.2k; footprint Resistor_SMD:R_0603_1608Metric_Pad1.05x0.95mm_HandSolder -> Resistor_SMD:R_0603_1608Metric
- R24: value 1k -> 2.2k; footprint Resistor_SMD:R_0603_1608Metric_Pad1.05x0.95mm_HandSolder -> Resistor_SMD:R_0603_1608Metric
- moved J8 116.2 mm to (186.3, 106.2), turned to 0 degrees
- moved J6 97.4 mm to (193.0, 106.2), turned to 0 degrees
- moved R24 94.6 mm to (155.1, 161.3), turned to 0 degrees
- moved C11 77.5 mm to (158.4, 156.5), turned to 0 degrees
- moved H1 73.0 mm to (132.9, 99.0)
- moved J1 72.1 mm to (162.0, 127.0)
- moved R9 71.3 mm to (37.8, 135.6)
- moved R8 71.3 mm to (37.9, 134.1)
- moved C2 71.0 mm to (38.8, 128.4)
- moved C3 71.0 mm to (35.7, 130.7)
- moved U2 71.0 mm to (37.7, 131.2)
- moved D1 70.6 mm to (39.8, 130.8)
- moved R22 70.2 mm to (151.5, 156.2), turned to 180 degrees
- moved R23 69.6 mm to (144.4, 161.3), turned to 0 degrees
- moved C12 68.6 mm to (93.0, 146.6)
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Connections:
- net EXP_TXD renamed ESP_TXD
- net IO4 renamed ESP_SD_CS
- C11 pad 1: Net-(AC1-Pad26) -> GND
- C11 pad 2: GND -> +3V3
- C6 pad 1: +3V3 -> Net-(C6-Pad1)
- C9 pad 1: Net-(AC1-Pad9) -> +3V3
- J1 pad 1: IO2 -> Net-(J1-Pad1)
- J1 pad 3: IO36 -> ESP_SPI_MOSI
- J1 pad 4: IO39 -> +3V3
- J6 pad 1: PS0\WAKE -> +3V3
- J6 pad 2: PS1 -> +3V3
- J7 pad 1: BOOT -> GND
- J8 pad 1: Resistive_Stretch_OUT -> Resistive_Stretch2
- J8 pad 2: +3V3 -> Resistive_Stretch1
- Q2 pad 1: Vibrator_MOTOR -> Vibrator_MOTOR2
- R10 pad 1: PS0\WAKE -> +3V3
- R10 pad 2: GND -> Net-(R10-Pad2)
- R11 pad 1: PS1 -> Net-(R10-Pad2)
- R11 pad 2: GND -> Capacitive_Stretch1
- R13 pad 2: BOOT -> Net-(R13-Pad2)
- R14 pad 1: RST -> Net-(R13-Pad2)
- R14 pad 2: +3V3 -> Capacitive_Stretch2
- R18 pad 1: +3V3 -> +1V8
- R18 pad 2: Net-(AC1-Pad15) -> IMU_CLK
- R20 pad 1: +3V3 -> +1V8
- R20 pad 2: Net-(AC1-Pad16) -> IMU_MOSI
- R21 pad 2: ADDR\MOSI -> ESP_SPI_CLK
- R22 pad 1: SCL\SCK\RX -> +3V3
- R22 pad 2: Net-(JP7-Pad1) -> ESP_SPI_MOSI
- R23 pad 1: SDA\MISO\TX -> +1V8
- R23 pad 2: Net-(JP7-Pad3) -> IMU_CS
- R24 pad 1: GND -> +1V8
- R24 pad 2: Resistive_Stretch_OUT -> IMU_MISO
- U1 pad 24: IO2 -> Buzzer_IN
- U1 pad 29: SPI_CS -> ESP_IMU_CS
- U1 pad 30: SPI_CLK -> ESP_SPI_CLK
- U1 pad 31: SPI_MISO -> ESP_SPI_MISO
- U1 pad 33: I2C_SDA -> Vibrator_MOTOR1
- U1 pad 36: I2C_SCL -> Vibrator_MOTOR2
- U1 pad 37: SPI_MOSI -> ESP_SPI_MOSI
- U1 pad 4: IO36 -> Capacitive_Stretch1_OUT
- U1 pad 5: IO39 -> Capacitive_Stretch2_OUT
- U1 pad 6: Resistive_Stretch_OUT -> Resistive_Stretch2
- U1 pad 8: INT -> Extern_Sensor
- U1 pad 9: Vibrator_MOTOR -> Resistive_Stretch1
Routing:
- net +3V3: track 246.4 -> 0.00 mm, vias 7 -> 0
- net +BATT: track 148.4 -> 0.00 mm, vias 2 -> 0
- net GND: track 70.0 -> 0.00 mm, vias 64 -> 0
- net INT: track 56.7 -> 0.00 mm, vias 4 -> 0
- net PS0\WAKE: track 50.7 -> 0.00 mm, vias 1 -> 0
- net SPI_CS: track 50.4 -> 0.00 mm, vias 3 -> 0
- net SCL\SCK\RX: track 46.1 -> 0.00 mm, vias 4 -> 0
- net SPI_MOSI: track 46.1 -> 0.00 mm, vias 1 -> 0
- net SDA\MISO\TX: track 40.2 -> 0.00 mm, vias 3 -> 0
- net ADDR\MOSI: track 38.8 -> 0.00 mm, vias 3 -> 0
- net I2C_SCL: track 36.4 -> 0.00 mm, vias 1 -> 0
- net RST: track 35.7 -> 0.00 mm, vias 3 -> 0
- net I2C_SDA: track 32.7 -> 0.00 mm, vias 1 -> 0
- net ESP_EN: track 30.9 -> 0.00 mm, vias 2 -> 0
- net ESP_IO0: track 29.9 -> 0.00 mm, vias 4 -> 0
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- removed copper zone on B.Cu, net GND
- removed copper zone on F.Cu, net GND
Other:
- board outline removed
- board text removed: "3.3V"
- board text removed: "B+"
- board text removed: "B-"
- board text removed: "CS"
- board text removed: "ESP_TXD"
- board text removed: "GND"
- board text removed: "INT"
- board text removed: "IO39"
- board text removed: "Kinetic-Analysis COPD Shirt PCB Versie 1.0"
- board text removed: "M+"
- board text removed: "M-"
- board text removed: "MISO"
- board text removed: "MOSI"
- board text removed: "PS0"
- board text removed: "PS1"
- board text removed: "R+"
- board text removed: "R-"
- board text removed: "RST"
- board text removed: "SCK"
- board text removed: "SCL"
- board text removed: "SDA"
- board text removed: "WAKE"

Commit message: KiCad New layout
Parts:
- removed Q9: Q_NMOS_GSD, Package_TO_SOT_SMD:SOT-23
- added BZ1: Buzzer, Buzzer_Beeper:Buzzer_TDK_PS1240P02BT_D12.2mm_H6.5mm, F.Cu at (107.6, 107.7)
- added J12: Conn_01x01_Male, Connector_PinHeader_2.54mm:PinHeader_1x01_P2.54mm_Vertical, F.Cu at (114.0, 87.7)
- added J13: Screw_Terminal_01x02, TerminalBlock_TE-Connectivity:TerminalBlock_TE_282834-2_1x02_P2.54mm_Horizontal, F.Cu at (104.0, 90.5)
- added J5: Conn_01x06_Male, Versie1_FootprintLib:IMU_Testpins, B.Cu at (93.0, 70.9)
- added JP1: SolderJumper_2_Open, Jumper:SolderJumper-2_P1.3mm_Open_Pad1.0x1.5mm, B.Cu at (100.9, 87.2)
- added JP10: SolderJumper_2_Open, Jumper:SolderJumper-2_P1.3mm_Open_Pad1.0x1.5mm, B.Cu at (72.9, 87.4)
- added JP2: SolderJumper_2_Open, Jumper:SolderJumper-2_P1.3mm_Open_Pad1.0x1.5mm, B.Cu at (91.6, 86.7)
- added JP3: SolderJumper_2_Open, Jumper:SolderJumper-2_P1.3mm_Open_Pad1.0x1.5mm, B.Cu at (93.0, 93.2)
- added JP4: SolderJumper_2_Open, Jumper:SolderJumper-2_P1.3mm_Open_Pad1.0x1.5mm, B.Cu at (85.2, 87.0)
- added JP5: SolderJumper_2_Open, Jumper:SolderJumper-2_P1.3mm_Open_Pad1.0x1.5mm, B.Cu at (75.8, 86.8)
- added JP6: SolderJumper_2_Open, Jumper:SolderJumper-2_P1.3mm_Open_Pad1.0x1.5mm, B.Cu at (77.5, 92.9)
- added JP7: SolderJumper_2_Open, Jumper:SolderJumper-2_P1.3mm_Open_Pad1.0x1.5mm, B.Cu at (88.6, 87.4)
- D2, D3: footprint Diode_SMD:D_1206_3216Metric_Pad1.42x1.75mm_HandSolder -> Diode_SMD:D_0603_1608Metric
- J1: value Micro_SD_Card -> Micro_SD_Card_Det; moved to B.Cu
- J3: footprint Connector_PinHeader_2.54mm:PinHeader_2x05_P2.54mm_Vertical -> Versie1_FootprintLib:Pin_Header_2x5_1.27mm_CONN
- J4: footprint Connector_PinHeader_2.54mm:PinHeader_2x03_P2.54mm_Vertical -> Versie1_FootprintLib:Pin_Header_2x3_1.27mm_CONN
- JP8, JP9: moved to B.Cu
- moved J6 133.2 mm to (70.4, 54.2), turned to 180 degrees
- moved R30 120.6 mm to (69.6, 86.2)
- moved J8 120.4 mm to (66.9, 90.5)
- moved R31 120.3 mm to (66.6, 86.2), turned to 180 degrees
- moved C15 108.2 mm to (102.3, 68.7), turned to 270 degrees
- moved R27 107.6 mm to (109.1, 51.3), turned to 90 degrees
- moved U5 107.5 mm to (99.9, 68.8), turned to 0 degrees
- moved C19 107.1 mm to (107.5, 71.5), turned to 90 degrees
- moved C11 106.9 mm to (97.5, 68.6), turned to 90 degrees
- moved C17 106.5 mm to (106.0, 71.5), turned to 90 degrees
- moved C18 105.9 mm to (104.4, 71.5), turned to 90 degrees
- moved R25 105.4 mm to (109.1, 54.7), turned to 90 degrees
- moved LED1 105.2 mm to (112.8, 57.8), turned to 180 degrees
- moved Q4 104.6 mm to (106.6, 51.2), turned to 90 degrees
- moved R24 103.7 mm to (102.5, 71.9), turned to 90 degrees
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Connections:
- C7 pad 1: +3V3 -> Net-(C7-Pad1)
- C9 pad 1: +3V3 -> Net-(C9-Pad1)
- IC1 pad 4: Net-(IC1-Pad4) -> (no net)
- IC1 pad 7: Net-(IC1-Pad7) -> (no net)
- IC2 pad 11: Net-(IC2-Pad11) -> (no net)
- J1 pad 1: Net-(J1-Pad1) -> (no net)
- J1 pad 11: (no net) -> GND
- J1 pad 8: Net-(J1-Pad8) -> (no net)
- J1 pad 9: GND -> (no net)
- J2 pad A5: Net-(J2-PadA5) -> (no net)
- J2 pad A6: Net-(J2-PadA6) -> (no net)
- J2 pad A7: Net-(J2-PadA7) -> (no net)
- J2 pad A8: Net-(J2-PadA8) -> (no net)
- J2 pad B5: Net-(J2-PadB5) -> (no net)
- J2 pad B6: Net-(J2-PadB6) -> (no net)
- J2 pad B7: Net-(J2-PadB7) -> (no net)
- J2 pad B8: Net-(J2-PadB8) -> (no net)
- J3 pad 1: +3V3 -> (no net)
- J3 pad 6: Net-(J3-Pad6) -> (no net)
- J4 pad 6: +3V3 -> (no net)
- R10 pad 1: +3V3 -> Net-(C7-Pad1)
- R11 pad 2: Capacitive_Stretch1 -> Net-(JP3-Pad1)
- R13 pad 1: +3V3 -> Net-(C9-Pad1)
- R14 pad 2: Capacitive_Stretch2 -> Net-(JP6-Pad1)
- R32 pad 1: Net-(BZ1-Pad2) -> GND
- R32 pad 2: +3V3 -> Piezo_Speaker
- U1 pad 10: Green_LED -> Piezo_Speaker
- U1 pad 11: Yellow_LED -> Vibrator_MOTOR2
- U1 pad 12: Red_LED -> Capacitive_Stretch1_OUT
- U1 pad 17: Net-(U1-Pad17) -> (no net)
- U1 pad 18: Net-(U1-Pad18) -> (no net)
- U1 pad 19: Net-(U1-Pad19) -> (no net)
- U1 pad 20: Net-(U1-Pad20) -> (no net)
- U1 pad 21: Net-(U1-Pad21) -> (no net)
- U1 pad 22: Net-(U1-Pad22) -> (no net)
- U1 pad 24: Buzzer_IN -> Touch_Pad
- U1 pad 27: uC_SENSE -> Yellow_LED
- U1 pad 28: uC_LATCH -> Green_LED
- U1 pad 32: Net-(U1-Pad32) -> (no net)
- U1 pad 33: Vibrator_MOTOR1 -> Red_LED
- U1 pad 36: Vibrator_MOTOR2 -> Vibrator_MOTOR1
- U1 pad 4: Capacitive_Stretch1_OUT -> Resistive_Stretch1
- U1 pad 5: Capacitive_Stretch2_OUT -> Resistive_Stretch2
- U1 pad 6: Resistive_Stretch2 -> uC_SENSE
- U1 pad 8: Extern_Sensor -> Capacitive_Stretch2_OUT
- U1 pad 9: Resistive_Stretch1 -> uC_LATCH
- U2 pad 7: Net-(U2-Pad7) -> (no net)
- U3 pad 2: Capacitive_Stretch1 -> Net-(JP3-Pad1)
- U3 pad 3: Capacitive_Stretch1_OUT -> Net-(JP2-Pad1)
- U3 pad 4: +3V3 -> Net-(C7-Pad1)
- U3 pad 6: Capacitive_Stretch1 -> Net-(JP3-Pad1)
- U3 pad 8: +3V3 -> Net-(C7-Pad1)
- U4 pad 2: Capacitive_Stretch2 -> Net-(JP6-Pad1)
- U4 pad 3: Capacitive_Stretch2_OUT -> Net-(JP5-Pad1)
- U4 pad 4: +3V3 -> Net-(C9-Pad1)
- U4 pad 6: Capacitive_Stretch2 -> Net-(JP6-Pad1)
- U4 pad 8: +3V3 -> Net-(C9-Pad1)
- U5 pad 4: Net-(U5-Pad4) -> (no net)
- U6 pad 1: Net-(U6-Pad1) -> (no net)
- U6 pad 11: Net-(U6-Pad11) -> (no net)
- U6 pad 12: Net-(U6-Pad12) -> (no net)
- U6 pad 14: Net-(U6-Pad14) -> (no net)
- U6 pad 15: Net-(U6-Pad15) -> (no net)
- U6 pad 16: Net-(U6-Pad16) -> (no net)
- U6 pad 17: Net-(U6-Pad17) -> (no net)
- U6 pad 19: Net-(U6-Pad19) -> (no net)
- U6 pad 2: Net-(U6-Pad2) -> (no net)
- U6 pad 21: Net-(U6-Pad21) -> (no net)
- U6 pad 3: Net-(U6-Pad3) -> (no net)
- U6 pad 4: Net-(U6-Pad4) -> (no net)
- U6 pad 5: Net-(U6-Pad5) -> (no net)
- U6 pad 6: Net-(U6-Pad6) -> (no net)
- U6 pad 7: Net-(U6-Pad7) -> (no net)
Routing:
- net GND: track 0.00 -> 105.9 mm, vias 0 -> 43
- net Resistive_Stretch2: track 0.00 -> 27.9 mm, vias 0 -> 2
- net +3V3: track 0.00 -> 27.7 mm, vias 0 -> 13
- net Resistive_Stretch1: track 0.00 -> 21.9 mm, vias 0 -> 2
- net +1V8: track 0.00 -> 20.1 mm, vias 0 -> 7
- net Capacitive_Stretch1_OUT: track 0.00 -> 17.6 mm, vias 0 -> 3
- net +BATT: track 0.00 -> 15.9 mm, vias 0 -> 8
- net Net-(C7-Pad1): track 0.00 -> 14.3 mm, vias 0 -> 2
- net Net-(C9-Pad1): track 0.00 -> 14.0 mm, vias 0 -> 2
- net DC-DC_ENABLE: track 0.00 -> 12.5 mm
- net IMU_MOSI: track 0.00 -> 12.0 mm, vias 0 -> 2
- net Capacitive_Stretch2_OUT: track 0.00 -> 11.4 mm, vias 0 -> 1
- net Net-(JP3-Pad1): track 0.00 -> 10.5 mm, vias 0 -> 1
- net ESP_IO0: track 0.00 -> 10.5 mm, vias 0 -> 2
- net Net-(JP6-Pad1): track 0.00 -> 10.4 mm, vias 0 -> 1
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- added copper zone on PWR, net +1V8
- added copper zone on PWR, net +3V3
- added copper zone on PWR, net +5V
- added copper zone on PWR, net +BATT
- added copper zone on GND, net GND
Other:
- board outline added: 55.5 x 44.7 mm
- copper layers 2 -> 4
- rule trace_min: 0.25 -> 0.2

Commit message: KiCad PCB Versie 2 af
Parts:
- removed BZ1: Buzzer, Buzzer_Beeper:Buzzer_TDK_PS1240P02BT_D12.2mm_H6.5mm
- removed H1, H3, H4: MountingHole, MountingHole:MountingHole_3.2mm_M3
- added F1: Polyfuse_Small, Fuse:Fuse_0402_1005Metric, F.Cu at (85.3, 57.6)
- moved J6 6.70 mm to (77.1, 53.6)
- moved J4 5.89 mm to (69.5, 54.6)
- moved R12 1.01 mm to (87.8, 57.0)
- moved C8 0.96 mm to (87.8, 55.5)
- moved BT1 0.63 mm to (83.1, 53.6)
- moved R5 0.09 mm to (94.5, 67.6)
Connections:
- BT1 pad 1: +BATT -> Batt_Before_Fuse
- C3 pad 1: +BATT -> Batt_Before_Fuse
- R12 pad 2: +BATT -> Batt_Before_Fuse
- U2 pad 3: +BATT -> Batt_Before_Fuse
- U2 pad 4: +BATT -> Batt_Before_Fuse
Routing:
- net Touch_Pad: track 0.00 -> 73.7 mm, vias 0 -> 3
- net ESP_SPI_MOSI: track 2.20 -> 59.2 mm, vias 0 -> 5
- net ESP_MTMS: track 0.00 -> 56.8 mm, vias 0 -> 4
- net ESP_SPI_CLK: track 2.20 -> 57.6 mm, vias 0 -> 4
- net ESP_SPI_MISO: track 2.20 -> 56.0 mm, vias 0 -> 2
- net ESP_SD_CS: track 0.00 -> 48.0 mm, vias 0 -> 3
- net Vibrator_MOTOR1: track 0.00 -> 46.3 mm, vias 0 -> 2
- net Piezo_Speaker: track 0.00 -> 40.0 mm, vias 0 -> 2
- net Red_LED: track 0.00 -> 38.6 mm, vias 0 -> 2
- net ESP_IMU_CS: track 2.20 -> 39.5 mm, vias 0 -> 2
- net Yellow_LED: track 0.00 -> 36.4 mm, vias 0 -> 2
- net Vibrator_MOTOR2: track 0.00 -> 30.5 mm, vias 0 -> 2
- net uC_SENSE: track 0.00 -> 30.2 mm, vias 0 -> 1
- net ESP_EN: track 3.65 -> 32.3 mm, vias 0 -> 2
- net Green_LED: track 0.00 -> 27.8 mm, vias 0 -> 2
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- added copper zone on PWR, net Batt_Before_Fuse
Other:
- board size 55.5 x 44.7 mm -> 56.3 x 45.4 mm
- board text added: "3V3"
- board text added: "BATT+"
- board text added: "BATT-"
- board text added: "CAP1+"
- board text added: "CAP1-"
- board text added: "CAP2+"
- board text added: "CAP2-"
- board text added: "CLK"
- board text added: "GND"
- board text added: "IMU_CS"
- board text added: "Kinetic-Analysis COPD Shirt V2.0 17-04-2021 Jacky Wong"
- board text added: "M1+"
- board text added: "M1-"
- board text added: "M2+"
- board text added: "M2-"
- board text added: "MISO"
- board text added: "MOSI"
- board text added: "PIEZO+"
- board text added: "PIEZO-"
- board text added: "RES1+"
- board text added: "RES2+"
- board text added: "TOUCH"

Commit message: BOMLIST
Parts:
- F1: footprint Fuse:Fuse_0402_1005Metric -> Fuse:Fuse_0603_1608Metric
- moved F1 0.53 mm to (84.8, 57.7)
Routing:
- net Red_LED: track 38.6 -> 39.9 mm, vias 2 -> 4
- net ESP_IO0: track 16.6 -> 15.9 mm
